File: gorthage-truck.kicad_pcb (KiCad board)
At the start: 2 copper layers, 342.9 x 85.7 mm, 164 parts, among them SW1 RotaryEncoder_Switch, U1 ATmega32U4-A, U2 SRV05-4, Y1 16MHz

Commit message: Add gitignore
Parts:
- SW1: footprint Keebio-Parts:RotaryEncoder_EC11-no-legs -> Keebio-Parts:RotaryEncoder_EC11
- U1: footprint Package_QFP:TQFP-44_10x10mm_P0.8mm -> s8erdude-keyboard-parts:QFN_TQFP-44_Combined
- moved U2 3.70 mm to (285.7, 37.4)
- moved R2 2.38 mm to (287.0, 41.2)
- moved R3 2.38 mm to (284.5, 41.2)
- moved C8 1.78 mm to (273.7, 28.3)
- moved R10 1.78 mm to (275.6, 28.3)
- moved CHASSIS1 1.70 mm to (278.6, 27.5)
- moved R8 1.57 mm to (274.3, 24.8)
- moved SW1 1.52 mm to (285.5, 38.8)
- moved R6 1.52 mm to (293.6, 24.8)
- moved USB1 1.51 mm to (285.8, 22.1)
- moved C5 0.65 mm to (274.8, 40.1)
Routing:
- net +5V: track 86.6 -> 105.1 mm
- net ROW4: track 185.6 -> 192.4 mm
- net GND: track 124.4 -> 130.6 mm
- net RE_B: track 31.1 -> 35.3 mm, vias 2 -> 1
- net ROW5: track 222.0 -> 225.2 mm
- net LED_2: track 32.6 -> 35.7 mm
- net COL8: track 134.5 -> 137.6 mm
- net Net-(R4-Pad2): track 3.10 -> 6.17 mm
- net ROW6: track 217.7 -> 220.7 mm
- net LED_1: track 26.9 -> 29.9 mm
- net Net-(R1-Pad2): track 33.8 -> 36.8 mm
- net COL5: track 289.5 -> 292.5 mm
- net COL3: track 342.7 -> 345.4 mm
- net COL7: track 363.2 -> 366.0 mm
- net Net-(U1-Pad42): track 0.00 -> 2.74 mm
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Other:
- net class Default: trace_width 0.25 -> 0.2
- board text added: "inspired by trashman designed by s8erdude"
- board text added: "ne ortho avail"
