File: gorthage-truck.sch (KiCad schematic (older format))
At the start: 164 parts, among them SW1 RotaryEncoder_Switch, U1 ATmega32U4-A, U2 SRV05-4, Y1 16MHz

Commit message: Add gitignore
Parts:
- C1, C2: LCSC (none) -> C1804
- C3: LCSC (none) -> C28323
- C4, C5, C6: LCSC (none) -> C49678
- C7: LCSC (none) -> C15850
- C8: LCSC (none) -> C1744
- D1, D10, D11, D12, D13, D14, D15, D16, D17, D18, D19, D2, D20, D21, D22, D23, D24, D25, D26, D27, D28, D29, D3, D30, D31, D32, D33, D34, D35, D36, D37, D38, D39, D4, D40, D41, D42, D43, D44, D45, D46, D47, D48, D49, D5, D50, D51, D52, D53, D54, D55, D56, D57, D58, D59, D6, D60, D61, D62, D63, D7, D8, D9: LCSC (none) -> C64898
- F1: LCSC (none) -> C261942
- R1, R4: LCSC (none) -> C17414
- R10: LCSC (none) -> C17514
- R2, R3: LCSC (none) -> C17561
- R5, R7, R9: LCSC (none) -> C26010
- R6, R8: LCSC (none) -> C27834
- U1: LCSC (none) -> C44854
- U2: LCSC (none) -> C85364
- USB1: LCSC (none) -> C165948
- Y1: LCSC (none) -> C13738
